Commit message: nicer worlds

File: urdf/sensors_sim.xacro (robot description, xacro)
@@ -3,33 +3,130 @@
   <xacro:arg name="robot_name" default=""/>
   <xacro:arg name="tf_prefix" default=""/>
-  <!-- Fake Sprayer Laser -->
-  <link name="/sprayer">
-    <collision>
+  <!-- Kinect v2 -->
+  <xacro:property name="kinect2_parent" value="base_link" />
+  <xacro:property name="kinect2_name" value="kinect2" />
+  <xacro:property name="kinect2_cam_px" value="0.80" /> #0.75
+  <xacro:property name="kinect2_cam_py" value="0.0" />
+  <xacro:property name="kinect2_cam_pz" value="1.75" /> #0.5
+  <xacro:property name="kinect2_cam_or" value="0.0" />
+  <xacro:property name="kinect2_cam_op" value="1.0472" />  #0.785 #0.392 #0.610
+  <xacro:property name="kinect2_cam_oy" value="0.0" />
+  <link name="${kinect2_name}_link">
+    <visual>
+      <geometry>
+        <mesh filename="package://kinect2_description/meshes/sensors/kinect2.dae"/>
+      </geometry>
+      <origin xyz="0.0 0 0" rpy="0 0 3.141592"/>
+    </visual>
+    <collision name="box_collision">
+      <geometry>
+        <box size=".1 .25 .06"/>
+      </geometry>
+      <contact_coefficients mu="0" kp="1000.0" kd="1.0"/>
+    </collision>
+    <inertial>
+      <mass value="1e-5" />
       <origin xyz="0 0 0" rpy="0 0 0"/>
-      <geometry>
-        <box size="0.1 0.1 0.1"/>
-      </geometry>
-    </collision>
-    <visual>
-      <geometry>
-        <box size="0.1 0.1 0.1"/>
-      </geometry>
-    </visual>
-    <inertial>
-      <mass value="1" />
       <inertia ixx="1e-6" ixy="0" ixz="0" iyy="1e-6" iyz="0" izz="1e-6" />
     </inertial>
-  </link>
-  <gazebo reference="/sprayer">
-    <material>Gazebo/Orange</material>
+ </link>
+  <joint name="${kinect2_name}_joint" type="fixed">
+    <parent link="/${kinect2_parent}"/>
+    <child link="${kinect2_name}_link"/>
+    <origin xyz="${kinect2_cam_px} ${kinect2_cam_py} ${kinect2_cam_pz}" rpy="${kinect2_cam_or} ${kinect2_cam_op} ${kinect2_cam_oy}"/>
+  </joint>
+  <link name="${kinect2_name}_rgb_optical_frame"/>
+  <joint name="${kinect2_name}_rgb_joint" type="fixed">
+    <parent link="${kinect2_name}_link"/>
+    <child link="${kinect2_name}_rgb_optical_frame"/>
+    <origin xyz="0.02 -0.01 0.00" rpy="-1.57 0 -1.57"/> #0.1 -0.01 0.016
+  </joint>
+  <gazebo reference="${kinect2_name}_link">
+    <sensor name="${kinect2_name}_camera" type="camera">
+      <always_on>true</always_on>
+      <update_rate>10.0</update_rate> #30.0
+      <camera name="${kinect2_name}_camera">
+        <horizontal_fov>${84.1*3.14/180.0}</horizontal_fov>
+        <image>
+          <width>640</width>
+          <height>480</height>
+          <format>R8G8B8</format>
+        </image>
+        <clip>
+          <near>0.02</near>
+          <far>10.0</far>
+        </clip>
+        <noise>
+          <type>gaussian</type>
+          <mean>0.0</mean>
+          <stddev>0.007</stddev>
+        </noise>
+      </camera>
+      <plugin name="${kinect2_name}_camera_controller" filename="libgazebo_ros_camera.so">
+        <alwaysOn>true</alwaysOn>
+        <updateRate>10.0</updateRate> #30.0
+        <cameraName>${kinect2_name}_camera</cameraName>
+        <imageTopicName>rgb/image_color_rect</imageTopicName>
+        <cameraInfoTopicName>rgb/camera_info</cameraInfoTopicName>
+        <frameName>${kinect2_name}_rgb_optical_frame</frameName>
+        <baseline>0.1</baseline>
+        <distortionK1>0.0</distortionK1>
+        <distortionK2>0.0</distortionK2>
+        <distortionK3>0.0</distortionK3>
+        <distortionT1>0.0</distortionT1>
+        <distortionT2>0.0</distortionT2>
+      </plugin>
+    </sensor>
   </gazebo>
-  <joint name="base_link_sprayer" type="fixed">
-    <parent link="/base_link"/>
-    <child link="/sprayer"/>
-    <axis xyz="1 0 0" />
-    <origin xyz="-0.45 0.000 0.5" rpy="0 0 0"/>
-  </joint>
+    <link name="${kinect2_name}_depth_optical_frame"/>
+    <joint name="${kinect2_name}_depth_joint" type="fixed">
+      <parent link="${kinect2_name}_link"/>
+      <child link="${kinect2_name}_depth_optical_frame"/>
+      <origin xyz="0.05 0.01 0.016" rpy="-1.57 0 -1.57"/>
+    </joint>
+    <gazebo reference="${kinect2_name}_link">
+      <sensor name="${kinect2_name}_sensor" type="depth">
+        <always_on>true</always_on>
+        <update_rate>10.0</update_rate> #30.0
+        <camera name="${kinect2_name}_sensor">
+          <horizontal_fov>${70.6*3.14/180.0}</horizontal_fov>
+          <image>
+            <width>512</width>
+            <height>424</height>
+            <format>L8</format>
+          </image>
+          <clip>
+            <near>0.1</near>
+            <far>10.0</far>
+          </clip>
+          <noise>
+            <type>gaussian</type>
+            <mean>0.0</mean>
+            <stddev>0.001</stddev>
+          </noise>
+        </camera>
+        <plugin name="${kinect2_name}_sensor_controller" filename="libgazebo_ros_openni_kinect.so">
+          <cameraName>${kinect2_name}_sensor</cameraName>
+          <alwaysOn>true</alwaysOn>
+          <updateRate>10.0</updateRate> #30.0
+          <imageTopicName>depth/image_ir_rect</imageTopicName>
+          <depthImageTopicName>depth/image_depth_rect</depthImageTopicName>
+          <pointCloudTopicName>depth/points</pointCloudTopicName>
+          <cameraInfoTopicName>ir/camera_info</cameraInfoTopicName>
+          <depthimagecamerainfotopicname>depth/camera_info</depthimagecamerainfotopicname>
+          <frameName>${kinect2_name}_depth_optical_frame</frameName>
+          <pointCloudCutoff>0.5</pointCloudCutoff>
+          <pointCloudCutoffMax>8.0</pointCloudCutoffMax>
+          <baseline>0.1</baseline>
+          <distortionK1>0.0</distortionK1>
+          <distortionK2>0.0</distortionK2>
+          <distortionK3>0.0</distortionK3>
+          <distortionT1>0.0</distortionT1>
+          <distortionT2>0.0</distortionT2>
+        </plugin>
+      </sensor>
+    </gazebo>
   <!-- Hokuyo Laser -->
-  <link name="/hokuyo">
+  <!--link name="/hokuyo">
     <collision>
       <origin xyz="0 0 0" rpy="0 0 0"/>
@@ -55,7 +152,7 @@
     <axis xyz="0 1 0" />
     <origin xyz="0.7025 0.005 0.66" rpy="0 0 0"/>
-  </joint>
+  </joint-->
   <!--hokuyo-->
-  <gazebo reference="/hokuyo">
+  <!--gazebo reference="/hokuyo">
     <sensor name="$(arg robot_name)hokuyo_sensor" type="ray">
       <pose>0 0 0 0 0 0</pose>
@@ -79,8 +176,4 @@
         <noise>
           <type>gaussian</type>
-          <!-- Noise parameters based on published spec for Hokuyo laser
-               achieving "+-30mm" accuracy at range < 10m.  A mean of 0.0m and
-               stddev of 0.01m will put 99.7% of samples within 0.03m of the true
-               reading. -->
           <mean>0.0</mean>
           <stddev>0.01</stddev>
@@ -92,7 +185,7 @@
       </plugin>
     </sensor>
-  </gazebo>
+  </gazebo-->
   <!-- Velodyne VLP16 -->
-  <xacro:property name="velodyne_origin">
+  <!--xacro:property name="velodyne_origin">
     <origin xyz="0 0 1.56" rpy="0 0 0" />
   </xacro:property>
@@ -110,5 +203,5 @@
   <xacro:property name="velodyne_min_angle" value="-${M_PI}" />
   <xacro:property name="velodyne_max_angle" value="${M_PI}" />
-  <xacro:property name="velodyne_gpu" value="false"/>
+  <xacro:property name="velodyne_gpu" value="false"/-->
 <!--
   <joint name="$(arg robot_name)_${velodyne_name}_base_mount_joint" type="fixed">
@@ -244,127 +337,3 @@
     </xacro:unless>
   </gazebo> -->
-  <!-- Kinect v2 -->
-  <xacro:property name="kinect2_parent" value="base_link" />
-  <xacro:property name="kinect2_name" value="kinect2" />
-  <xacro:property name="kinect2_cam_px" value="0.80" /> #0.75
-  <xacro:property name="kinect2_cam_py" value="0.0" />
-  <xacro:property name="kinect2_cam_pz" value="1.75" /> #0.5
-  <xacro:property name="kinect2_cam_or" value="0.0" />
-  <xacro:property name="kinect2_cam_op" value="1.0472" />  #0.785 #0.392 #${M_PI/2}i #0.610
-  <xacro:property name="kinect2_cam_oy" value="0.0" /> #${-M_PI/2}
-  <link name="${kinect2_name}_link">
-    <visual>
-      <geometry>
-        <mesh filename="package://kinect2_description/meshes/sensors/kinect2.dae"/>
-      </geometry>
-      <origin xyz="0.0 0 0" rpy="0 0 3.141592"/>
-    </visual>
-    <collision name="box_collision">
-      <geometry>
-        <box size=".1 .25 .06"/>
-      </geometry>
-      <contact_coefficients mu="0" kp="1000.0" kd="1.0"/>
-    </collision>
-    <inertial>
-      <mass value="1e-5" />
-      <origin xyz="0 0 0" rpy="0 0 0"/>
-      <inertia ixx="1e-6" ixy="0" ixz="0" iyy="1e-6" iyz="0" izz="1e-6" />
-    </inertial>
- </link>
-  <joint name="${kinect2_name}_joint" type="fixed">
-    <parent link="/${kinect2_parent}"/>
-    <child link="${kinect2_name}_link"/>
-    <origin xyz="${kinect2_cam_px} ${kinect2_cam_py} ${kinect2_cam_pz}" rpy="${kinect2_cam_or} ${kinect2_cam_op} ${kinect2_cam_oy}"/>
-  </joint>
-  <link name="${kinect2_name}_rgb_optical_frame"/>
-  <joint name="${kinect2_name}_rgb_joint" type="fixed">
-    <parent link="${kinect2_name}_link"/>
-    <child link="${kinect2_name}_rgb_optical_frame"/>
-    <origin xyz="0.02 -0.01 0.00" rpy="-1.57 0 -1.57"/> #0.1 -0.01 0.016
-  </joint>
-  <!-- <link name="${kinect2_name}_depth_optical_frame"/>
-  <joint name="${kinect2_name}_depth_joint" type="fixed">
-    <parent link="${kinect2_name}_link"/>
-    <child link="${kinect2_name}_depth_optical_frame"/>
-    <origin xyz="0.05 0.01 0.016" rpy="-1.57 0 -1.57"/>
-  </joint> -->
-  <!-- <gazebo reference="${kinect2_name}_link">
-    <sensor name="${kinect2_name}_sensor" type="depth">
-      <always_on>true</always_on>
-      <update_rate>10.0</update_rate> #30.0
-      <camera name="${kinect2_name}_sensor">
-        <horizontal_fov>${70.6*3.14/180.0}</horizontal_fov>
-        <image>
-          <width>512</width>
-          <height>424</height>
-          <format>L8</format>
-        </image>
-        <clip>
-          <near>0.1</near>
-          <far>10.0</far>
-        </clip>
-        <noise>
-          <type>gaussian</type>
-          <mean>0.0</mean>
-          <stddev>0.001</stddev>
-        </noise>
-      </camera>
-      <plugin name="${kinect2_name}_sensor_controller" filename="libgazebo_ros_openni_kinect.so">
-        <cameraName>${kinect2_name}_sensor</cameraName>
-        <alwaysOn>true</alwaysOn>
-        <updateRate>10.0</updateRate> #30.0
-        <imageTopicName>depth/image_ir_rect</imageTopicName>
-        <depthImageTopicName>depth/image_depth_rect</depthImageTopicName>
-        <pointCloudTopicName>depth/points</pointCloudTopicName>
-        <cameraInfoTopicName>ir/camera_info</cameraInfoTopicName>
-        <depthimagecamerainfotopicname>depth/camera_info</depthimagecamerainfotopicname>
-        <frameName>${kinect2_name}_depth_optical_frame</frameName>
-        <pointCloudCutoff>0.5</pointCloudCutoff>
-        <pointCloudCutoffMax>8.0</pointCloudCutoffMax>
-        <baseline>0.1</baseline>
-        <distortionK1>0.0</distortionK1>
-        <distortionK2>0.0</distortionK2>
-        <distortionK3>0.0</distortionK3>
-        <distortionT1>0.0</distortionT1>
-        <distortionT2>0.0</distortionT2>
-      </plugin>
-    </sensor>
-  </gazebo> -->
-  <gazebo reference="${kinect2_name}_link">
-    <sensor name="${kinect2_name}_camera" type="camera">
-      <always_on>true</always_on>
-      <update_rate>10.0</update_rate> #30.0
-      <camera name="${kinect2_name}_camera">
-        <horizontal_fov>${84.1*3.14/180.0}</horizontal_fov>
-        <image>
-          <width>1920</width>
-          <height>1080</height>
-          <format>R8G8B8</format>
-        </image>
-        <clip>
-          <near>0.02</near>
-          <far>10.0</far>
-        </clip>
-        <noise>
-          <type>gaussian</type>
-          <mean>0.0</mean>
-          <stddev>0.007</stddev>
-        </noise>
-      </camera>
-      <plugin name="${kinect2_name}_camera_controller" filename="libgazebo_ros_camera.so">
-        <alwaysOn>true</alwaysOn>
-        <updateRate>10.0</updateRate> #30.0
-        <cameraName>${kinect2_name}_camera</cameraName>
-        <imageTopicName>rgb/image_color_rect</imageTopicName>
-        <cameraInfoTopicName>rgb/camera_info</cameraInfoTopicName>
-        <frameName>${kinect2_name}_rgb_optical_frame</frameName>
-        <baseline>0.1</baseline>
-        <distortionK1>0.0</distortionK1>
-        <distortionK2>0.0</distortionK2>
-        <distortionK3>0.0</distortionK3>
-        <distortionT1>0.0</distortionT1>
-        <distortionT2>0.0</distortionT2>
-      </plugin>
-    </sensor>
-  </gazebo>
 </robot>
